Commit message: Fixing issue with visp_auto_tracker package.

File: src/turtlebot3/turtlebot3_description/urdf/turtlebot3_waffle.urdf.xacro (robot description, xacro)
@@ -45,5 +45,5 @@
     <origin xyz="0 0 0" rpy="0 0 0"/>
     <geometry>
-      <mesh filename="package://turtlebot3_description/meshes/markers/QrCodeCube.dae" scale="0.3 0.3 0.3"/>
+      <mesh filename="package://turtlebot3_description/meshes/markers/MarkerCube.dae" scale="0.3 0.3 0.3"/>
     </geometry>
   </visual>
